Commit message: create moveit from MSA

File: src/ur5e_gripper/ur5e_gripper_description/urdf/ur5e_gripper.urdf.xacro (robot description, xacro)
@@ -49,10 +49,11 @@
   <!-- convert to property to use substitution in function -->
   <xacro:property name="initial_positions_file" default="$(arg initial_positions_file)"/>
+  <xacro:arg name="parent_link" default="world"/>
   <!-- create link fixed to the "world" -->
-  <link name="world" />
+  <link name="$(arg parent_link)" />
   <!-- arm -->
   <xacro:ur_robot name="$(arg name)"
     tf_prefix="$(arg tf_prefix)"
-    parent="world"
+    parent="$(arg parent_link)"
     joint_limits_parameters_file="$(arg joint_limit_params)"
     kinematics_parameters_file="$(arg kinematics_params)"
