Commit message: fix but not exactly fix

File: src/ur5e_gripper/robotiq_description/urdf/robotiq_2f_85_macro.urdf.xacro (robot description, xacro)
@@ -261,4 +261,26 @@
             <mimic joint="${prefix}robotiq_85_left_knuckle_joint" />
         </joint>
+        <!-- https://github.com/ros-controls/gazebo_ros2_control/issues/173 -->
+        <link name="dummy_child"/>
+        <joint name="${prefix}robotiq_85_right_knuckle_joint_mimic" type="fixed">
+            <parent link="${prefix}robotiq_85_base_link" />
+            <child link="dummy_child" />
+        </joint>
+        <joint name="${prefix}robotiq_85_left_inner_knuckle_joint_mimic" type="fixed">
+            <parent link="${prefix}robotiq_85_base_link" />
+            <child link="dummy_child" />
+        </joint>
+        <joint name="${prefix}robotiq_85_right_inner_knuckle_joint_mimic" type="fixed">
+            <parent link="${prefix}robotiq_85_base_link" />
+            <child link="dummy_child" />
+        </joint>
+        <joint name="${prefix}robotiq_85_left_finger_tip_joint_mimic" type="fixed">
+            <parent link="${prefix}robotiq_85_base_link" />
+            <child link="dummy_child" />
+        </joint>
+        <joint name="${prefix}robotiq_85_right_finger_tip_joint_mimic" type="fixed">
+            <parent link="${prefix}robotiq_85_base_link" />
+            <child link="dummy_child" />
+        </joint>
     </xacro:macro>
 </robot>

File: src/ur5e_gripper/ur5e_gripper_description/urdf/ur5e_gripper.urdf (robot description, URDF)
Before this commit: robot ur5e_gripper, 22 links, 21 joints
Links:
- removed link base_link0
- added link dummy_child
- added link world
Joints:
- added joint robotiq_85_left_finger_tip_joint_mimic: type continuous, parent robotiq_85_base_link, child dummy_child
- added joint robotiq_85_left_inner_knuckle_joint_mimic: type continuous, parent robotiq_85_base_link, child dummy_child
- added joint robotiq_85_right_finger_tip_joint_mimic: type continuous, parent robotiq_85_base_link, child dummy_child
- added joint robotiq_85_right_inner_knuckle_joint_mimic: type continuous, parent robotiq_85_base_link, child dummy_child
- added joint robotiq_85_right_knuckle_joint_mimic: type continuous, parent robotiq_85_base_link, child dummy_child
- joint base_joint: parent base_link0 -> world

Commit message: fix _mimic joint not found in moveit

File: src/ur5e_gripper/robotiq_description/urdf/robotiq_2f_85_macro.urdf.xacro (robot description, xacro)
@@ -262,24 +262,28 @@
         </joint>
         <!-- https://github.com/ros-controls/gazebo_ros2_control/issues/173 -->
-        <link name="dummy_child"/>
+        <link name="dummy_child1"/>
+        <link name="dummy_child2"/>
+        <link name="dummy_child3"/>
+        <link name="dummy_child4"/>
+        <link name="dummy_child5"/>
         <joint name="${prefix}robotiq_85_right_knuckle_joint_mimic" type="fixed">
             <parent link="${prefix}robotiq_85_base_link" />
-            <child link="dummy_child" />
+            <child link="dummy_child1" />
         </joint>
         <joint name="${prefix}robotiq_85_left_inner_knuckle_joint_mimic" type="fixed">
             <parent link="${prefix}robotiq_85_base_link" />
-            <child link="dummy_child" />
+            <child link="dummy_child2" />
         </joint>
         <joint name="${prefix}robotiq_85_right_inner_knuckle_joint_mimic" type="fixed">
             <parent link="${prefix}robotiq_85_base_link" />
-            <child link="dummy_child" />
+            <child link="dummy_child3" />
         </joint>
         <joint name="${prefix}robotiq_85_left_finger_tip_joint_mimic" type="fixed">
             <parent link="${prefix}robotiq_85_base_link" />
-            <child link="dummy_child" />
+            <child link="dummy_child4" />
         </joint>
         <joint name="${prefix}robotiq_85_right_finger_tip_joint_mimic" type="fixed">
             <parent link="${prefix}robotiq_85_base_link" />
-            <child link="dummy_child" />
+            <child link="dummy_child5" />
         </joint>
     </xacro:macro>

File: src/ur5e_gripper/ur5e_gripper_description/urdf/ur5e_gripper.urdf (robot description, URDF)
Before this commit: robot ur5e_gripper, 23 links, 26 joints
Links:
- removed link dummy_child
- added link dummy_child1
- added link dummy_child2
- added link dummy_child3
- added link dummy_child4
- added link dummy_child5
Joints:
- joint robotiq_85_left_finger_tip_joint_mimic: child dummy_child -> dummy_child4; type continuous -> fixed
- joint robotiq_85_left_inner_knuckle_joint_mimic: child dummy_child -> dummy_child2; type continuous -> fixed
- joint robotiq_85_right_finger_tip_joint_mimic: child dummy_child -> dummy_child5; type continuous -> fixed
- joint robotiq_85_right_inner_knuckle_joint_mimic: child dummy_child -> dummy_child3; type continuous -> fixed
- joint robotiq_85_right_knuckle_joint_mimic: child dummy_child -> dummy_child1; type continuous -> fixed

Commit message: dual arms visualization and gazebo

File: src/ur5e_gripper/robotiq_description/urdf/robotiq_2f_85_macro.urdf.xacro (robot description, xacro)
@@ -262,28 +262,28 @@
         </joint>
         <!-- https://github.com/ros-controls/gazebo_ros2_control/issues/173 -->
-        <link name="dummy_child1"/>
-        <link name="dummy_child2"/>
-        <link name="dummy_child3"/>
-        <link name="dummy_child4"/>
-        <link name="dummy_child5"/>
+        <link name="${prefix}dummy_child1"/>
+        <link name="${prefix}dummy_child2"/>
+        <link name="${prefix}dummy_child3"/>
+        <link name="${prefix}dummy_child4"/>
+        <link name="${prefix}dummy_child5"/>
         <joint name="${prefix}robotiq_85_right_knuckle_joint_mimic" type="fixed">
             <parent link="${prefix}robotiq_85_base_link" />
-            <child link="dummy_child1" />
+            <child link="${prefix}dummy_child1" />
         </joint>
         <joint name="${prefix}robotiq_85_left_inner_knuckle_joint_mimic" type="fixed">
             <parent link="${prefix}robotiq_85_base_link" />
-            <child link="dummy_child2" />
+            <child link="${prefix}dummy_child2" />
         </joint>
         <joint name="${prefix}robotiq_85_right_inner_knuckle_joint_mimic" type="fixed">
             <parent link="${prefix}robotiq_85_base_link" />
-            <child link="dummy_child3" />
+            <child link="${prefix}dummy_child3" />
         </joint>
         <joint name="${prefix}robotiq_85_left_finger_tip_joint_mimic" type="fixed">
             <parent link="${prefix}robotiq_85_base_link" />
-            <child link="dummy_child4" />
+            <child link="${prefix}dummy_child4" />
         </joint>
         <joint name="${prefix}robotiq_85_right_finger_tip_joint_mimic" type="fixed">
             <parent link="${prefix}robotiq_85_base_link" />
-            <child link="dummy_child5" />
+            <child link="${prefix}dummy_child5" />
         </joint>
     </xacro:macro>
