Commit message: test dual moveit control

File: src/ur5e_gripper/dual_ur5e_gripper_moveit_config/urdf/dual_ur5e_gripper.urdf.xacro (robot description, xacro)
@@ -9,9 +9,9 @@
     <!-- Left arm -->
     <xacro:ur5e_gripper name="left_ur" prefix="left_" parent="world" initial_positions_file="$(arg left_initial_positions_file)">
-        <origin xyz="0 -0.5 0" rpy="0 0 0" />
+        <origin xyz="0 0.5 0" rpy="0 0 0" />
     </xacro:ur5e_gripper>
     <!-- Right arm -->
     <xacro:ur5e_gripper name="right_ur" prefix="right_" parent="world" initial_positions_file="$(arg right_initial_positions_file)">
-        <origin xyz="0 0.5 0" rpy="0 0 0" />
+        <origin xyz="0 -0.5 0" rpy="0 0 0" />
     </xacro:ur5e_gripper>
     <gazebo>

Commit message: dd

File: src/ur5e_gripper/dual_ur5e_gripper_moveit_config/urdf/dual_ur5e_gripper.urdf.xacro (robot description, xacro)
@@ -9,9 +9,9 @@
     <!-- Left arm -->
     <xacro:ur5e_gripper name="left_ur" prefix="left_" parent="world" initial_positions_file="$(arg left_initial_positions_file)">
-        <origin xyz="0 0.5 0" rpy="0 0 0" />
+        <origin xyz="0 0.5 1.03" rpy="0 0 0" />
     </xacro:ur5e_gripper>
     <!-- Right arm -->
     <xacro:ur5e_gripper name="right_ur" prefix="right_" parent="world" initial_positions_file="$(arg right_initial_positions_file)">
-        <origin xyz="0 -0.5 0" rpy="0 0 0" />
+        <origin xyz="0 -0.5 1.03" rpy="0 0 0" />
     </xacro:ur5e_gripper>
     <gazebo>

Commit message: realsense in gazebo

File: src/ur5e_gripper/dual_ur5e_gripper_moveit_config/urdf/dual_ur5e_gripper.urdf.xacro (robot description, xacro)
@@ -15,4 +15,12 @@
         <origin xyz="0 -0.5 1.03" rpy="0 0 0" />
     </xacro:ur5e_gripper>
+    <!-- realsense d435 -->
+    <xacro:arg name="use_nominal_extrinsics" default="true"/>
+    <xacro:arg name="add_plug" default="false" />
+    <xacro:arg name="use_mesh" default="true" />
+    <xacro:include filename="$(find realsense2_description)/urdf/_d435.urdf.xacro" />
+    <xacro:sensor_d435 parent="world" use_nominal_extrinsics="$(arg use_nominal_extrinsics)" add_plug="$(arg add_plug)" use_mesh="$(arg use_mesh)">
+        <origin xyz="0.4 0 3.0" rpy="0 1.5707 0"/>
+    </xacro:sensor_d435>
     <gazebo>
         <plugin filename="libgazebo_ros2_control.so" name="gazebo_ros2_control">

Commit message: rewrite obj_detect.py but still has bug

File: src/ur5e_gripper/dual_ur5e_gripper_moveit_config/urdf/dual_ur5e_gripper.urdf.xacro (robot description, xacro)
@@ -21,5 +21,5 @@
     <xacro:include filename="$(find realsense2_description)/urdf/_d435.urdf.xacro" />
     <xacro:sensor_d435 parent="world" use_nominal_extrinsics="$(arg use_nominal_extrinsics)" add_plug="$(arg add_plug)" use_mesh="$(arg use_mesh)">
-        <origin xyz="0.4 0 3.0" rpy="0 1.5707 0"/>
+        <origin xyz="2 0 2.5" rpy="0 0.785398163 3.1415926"/>
     </xacro:sensor_d435>
     <gazebo>

Commit message: can detect obj and depth image is available now

File: src/ur5e_gripper/dual_ur5e_gripper_moveit_config/urdf/dual_ur5e_gripper.urdf.xacro (robot description, xacro)
@@ -21,5 +21,5 @@
     <xacro:include filename="$(find realsense2_description)/urdf/_d435.urdf.xacro" />
     <xacro:sensor_d435 parent="world" use_nominal_extrinsics="$(arg use_nominal_extrinsics)" add_plug="$(arg add_plug)" use_mesh="$(arg use_mesh)">
-        <origin xyz="2 0 2.5" rpy="0 0.785398163 3.1415926"/>
+        <origin xyz="1.5 0 2" rpy="0 0.785398163 3.1415926"/>
     </xacro:sensor_d435>
     <gazebo>
