Commit message: coordinate broadcast

File: src/ur5e_gripper/dual_ur5e_gripper_moveit_config/urdf/test.urdf (robot description, URDF)
Before this commit: robot dual_ur5e_gripper, 53 links, 52 joints
Links:
- added link camera_bottom_screw_frame
- added link camera_color_frame
- added link camera_color_optical_frame
- added link camera_depth_frame
- added link camera_depth_optical_frame
- added link camera_infra1_frame
- added link camera_infra1_optical_frame
- added link camera_infra2_frame
- added link camera_infra2_optical_frame
- added link camera_link, mass 0.072; collision box size=0.02505 0.09 0.025; visual mesh filename=file:///home/xiaobaige/UR5e_Vision_Assemble/install/realsen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
Joints:
- added joint camera_color_joint: type fixed, parent camera_link, child camera_color_frame, origin xyz=0 0.015 0 rpy=0 0 0
- added joint camera_color_optical_joint: type fixed, parent camera_color_frame, child camera_color_optical_frame, origin xyz=0 0 0 rpy=-1.5707963267948966 0 -1.5707963267948966
- added joint camera_depth_joint: type fixed, parent camera_link, child camera_depth_frame, origin xyz=0 0 0 rpy=0 0 0
- added joint camera_depth_optical_joint: type fixed, parent camera_depth_frame, child camera_depth_optical_frame, origin xyz=0 0 0 rpy=-1.5707963267948966 0 -1.5707963267948966
- added joint camera_infra1_joint: type fixed, parent camera_link, child camera_infra1_frame, origin xyz=0 0.0 0 rpy=0 0 0
- added joint camera_infra1_optical_joint: type fixed, parent camera_infra1_frame, child camera_infra1_optical_frame, origin xyz=0 0 0 rpy=-1.5707963267948966 0 -1.5707963267948966
- added joint camera_infra2_joint: type fixed, parent camera_link, child camera_infra2_frame, origin xyz=0 -0.05 0 rpy=0 0 0
- added joint camera_infra2_optical_joint: type fixed, parent camera_infra2_frame, child camera_infra2_optical_frame, origin xyz=0 0 0 rpy=-1.5707963267948966 0 -1.5707963267948966
- added joint camera_joint: type fixed, parent world, child camera_bottom_screw_frame, origin xyz=1.5 0 2 rpy=0 0.785398163 3.1415926
- added joint camera_link_joint: type fixed, parent camera_bottom_screw_frame, child camera_link, origin xyz=0.010600000000000002 0.0175 0.0125 rpy=0 0 0
- joint left_base_joint: origin xyz=0 -0.5 0 rpy=0 0 0 -> xyz=0 0.5 1.03 rpy=0 0 0
- joint right_base_joint: origin xyz=0 0.5 0 rpy=0 0 0 -> xyz=0 -0.5 1.03 rpy=0 0 0
