Commit message: can grasp

File: src/ur5e_gripper/dual_ur5e_gripper_moveit_config/srdf/dual_ur5e_gripper.srdf.xacro (robot description, xacro)
@@ -11,4 +11,20 @@
         <group name="right_ur_manipulator"/>
     </group>
+    <group_state name="left_ready" group="left_ur_manipulator">
+        <joint name="left_elbow_joint" value="1.5707" />
+        <joint name="left_shoulder_lift_joint" value="-1.5707" />
+        <joint name="left_shoulder_pan_joint" value="0" />
+        <joint name="left_wrist_1_joint" value="-1.5707" />
+        <joint name="left_wrist_2_joint" value="-1.5707" />
+        <joint name="left_wrist_3_joint" value="0" />
+    </group_state>
+    <group_state name="right_home" group="right_ur_manipulator">
+        <joint name="right_elbow_joint" value="1.5707" />
+        <joint name="right_shoulder_lift_joint" value="-1.5707" />
+        <joint name="right_shoulder_pan_joint" value="0" />
+        <joint name="right_wrist_1_joint" value="-1.5707" />
+        <joint name="right_wrist_2_joint" value="-1.5707" />
+        <joint name="right_wrist_3_joint" value="0" />
+      </group_state>
     <disable_collisions link1="left_robotiq_85_base_link" link2="left_wrist_1_link" reason="Never"/>
     <disable_collisions link1="left_robotiq_85_base_link" link2="left_wrist_2_link" reason="Never"/>

File: src/ur5e_gripper/dual_ur5e_gripper_moveit_config/urdf/dual_ur5e_gripper.urdf.xacro (robot description, xacro)
@@ -55,9 +55,9 @@
             </arm>
             <forces_angle_tolerance>150</forces_angle_tolerance>
-            <update_rate>50</update_rate>
-            <grip_count_threshold>2</grip_count_threshold>
-            <max_grip_count>8</max_grip_count>
-            <release_tolerance>0.05</release_tolerance>
-            <disable_collisions_on_attach>true</disable_collisions_on_attach>
+            <update_rate>30</update_rate>
+            <grip_count_threshold>1</grip_count_threshold>
+            <max_grip_count>2</max_grip_count>
+            <release_tolerance>0.01</release_tolerance>
+            <disable_collisions_on_attach>false</disable_collisions_on_attach>
             <contact_topic>__default_topic__</contact_topic>
          </plugin>
